Commit message: iteration 1

File: hivemind_env/assets/diff_drive_bot.urdf (robot description, URDF)
Before this commit: robot diff_drive_bot, 6 links, 5 joints
Links:
- added link arm_base_link, mass 0.1; visual cylinder length=0.012 radius=0.022
- added link arm_boom_link, mass 0.05; visual box size=0.10 0.016 0.012
- added link gripper_palm_link, mass 0.03; visual box size=0.012 0.07 0.012
- added link left_finger_link, mass 0.01; visual box size=0.05 0.008 0.014
- added link lidar_post_link, mass 0.02; visual cylinder length=0.07 radius=0.006
- added link right_finger_link, mass 0.01; visual box size=0.05 0.008 0.014
Joints:
- added joint arm_boom_joint: type fixed, parent arm_base_link, child arm_boom_link, origin xyz=0 0 0.005 rpy=0 0 0
- added joint arm_yaw_joint: type revolute, parent base_link, child arm_base_link, origin xyz=0 0 0.07 rpy=0 0 0, axis 0 0 1, limit lower=-3.14159265 upper=3.14159265 effort=10.0 velocity=5.0
- added joint gripper_palm_joint: type fixed, parent arm_boom_link, child gripper_palm_link, origin xyz=0.10 0 0 rpy=0 0 0
- added joint left_finger_joint: type prismatic, parent gripper_palm_link, child left_finger_link, origin xyz=0 0.03 0 rpy=0 0 0, axis 0 1 0, limit lower=-0.02 upper=0.02 effort=5.0 velocity=1.0
- added joint lidar_post_joint: type fixed, parent base_link, child lidar_post_link, origin xyz=0 0 0.066 rpy=0 0 0
- added joint right_finger_joint: type prismatic, parent gripper_palm_link, child right_finger_link, origin xyz=0 -0.03 0 rpy=0 0 0, axis 0 1 0, limit lower=-0.02 upper=0.02 effort=5.0 velocity=1.0
- joint lidar_joint: axis (none) -> 0 0 1; limit (none) -> lower=0.0 upper=0.07 effort=10.0 velocity=1.0; type fixed -> prismatic
